File: preamp.brd (EAGLE design)
At the start: 53.3 x 47 mm, 27 parts, among them IC1 TL074P

Commit message: corrected audio jack drill sizes, added test points.
Parts:
- added LEFT_IN, LEFT_OUT, MIX_OUT, RIGHT_IN, RIGHT_OUT, TEST_GND, TEST_GND1, TIP: TEST_POINTMINIATURE, Keystone:PLATED_HOLE_1.02MM
- moved COUT 1.27 mm to (47.0, 48.3)
- moved U$5 1.27 mm to (25.4, 38.1)
Connections:
- net GND: now also TEST_GND.1, TEST_GND1.1
- net LEFT_IN: now also LEFT_IN.1
- net N$12: now also RIGHT_OUT.1
- net N$13: now also MIX_OUT.1
- net N$14: now also TIP.1
- net N$8: now also LEFT_OUT.1
- net RIGHT_IN: now also RIGHT_IN.1
Routing:
- net GND: track 99.5 -> 125.0 mm
- net N$8: track 34.7 -> 43.5 mm
- net N$13: track 31.2 -> 37.4 mm
- net N$12: track 28.2 -> 32.6 mm
- net LEFT_IN: track 11.1 -> 15.3 mm
- net N$14: track 19.0 -> 22.4 mm
- net N$3: track 40.3 -> 37.4 mm
- net RIGHT_IN: track 6.03 -> 8.69 mm
- net N$15: track 22.8 -> 23.4 mm
Other:
- board text added: "7 Apr 2018"
- board text added: "GND"
- board text added: "L"
- board text added: "R"
- board text added: "version 2"
- board text removed: "24 March 2018"
- board text removed: "version 1"
