File: preamp.sch (EAGLE design)
At the start: 23 parts, among them IC1 TL074P

Commit message: corrected audio jack drill sizes, added test points.
Parts:
- added LEFT_IN, LEFT_OUT, MIX_OUT, RIGHT_IN, RIGHT_OUT, TEST_GND, TEST_GND1, TIP: TEST_POINTMINIATURE, Keystone:TEST_POINTMINIATURE
Connections:
- net GND: now also TEST_GND.P$1, TEST_GND1.P$1
- net LEFT_IN: now also LEFT_IN.P$1
- net N$12: now also RIGHT_OUT.P$1
- net N$13: now also MIX_OUT.P$1
- net N$14: now also TIP.P$1
- net N$8: now also LEFT_OUT.P$1
- net RIGHT_IN: now also RIGHT_IN.P$1
Other:
- moved on the sheet: C3, C4
Changed lines of the file:
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@@
 <part name="U$5" library="Bourns" deviceset="POTENTIOMETER" device="3362P"/>
 <part name="COUT" library="KEMET" deviceset="CAP" device="" value="2.2u"/>
+<part name="LEFT_IN" library="Keystone" deviceset="TEST_POINT" device="MINIATURE"/>
+<part name="RIGHT_IN" library="Keystone" deviceset="TEST_POINT" device="MINIATURE"/>
+<part name="LEFT_OUT" library="Keystone" deviceset="TEST_POINT" device="MINIATURE"/>
+<part name="RIGHT_OUT" library="Keystone" deviceset="TEST_POINT" device="MINIATURE"/>
+<part name="MIX_OUT" library="Keystone" deviceset="TEST_POINT" device="MINIATURE"/>
+<part name="TIP" library="Keystone" deviceset="TEST_POINT" device="MINIATURE"/>
+<part name="TEST_GND" library="Keystone" deviceset="TEST_POINT" device="MINIATURE"/>
+<part name="GND8" library="SparkFun-Aesthetics" deviceset="GND" device=""/>
+<part name="TEST_GND1" library="Keystone" deviceset="TEST_POINT" device="MINIATURE"/>
+<part name="GND9" library="SparkFun-Aesthetics" deviceset="GND" device=""/>
 </parts>
 <sheets>
@@
 <instance part="GND1" gate="1" x="-5.08" y="50.8"/>
 <instance part="GND2" gate="1" x="-7.62" y="7.62"/>
-<instance part="C3" gate="G$1" x="58.42" y="53.34"/>
-<instance part="C4" gate="G$1" x="58.42" y="30.48"/>
+<instance part="C3" gate="G$1" x="60.96" y="53.34"/>
+<instance part="C4" gate="G$1" x="60.96" y="30.48"/>
 <instance part="LMG" gate="G$1" x="66.04" y="60.96"/>
 <instance part="RMG" gate="G$1" x="66.04" y="38.1"/>
@@
 <instance part="U$5" gate="G$1" x="99.06" y="66.04"/>
 <instance part="COUT" gate="G$1" x="119.38" y="33.02"/>
+<instance part="LEFT_IN" gate="G$1" x="2.54" y="71.12"/>
+<instance part="RIGHT_IN" gate="G$1" x="2.54" y="48.26"/>
+<instance part="LEFT_OUT" gate="G$1" x="55.88" y="53.34"/>
+<instance part="RIGHT_OUT" gate="G$1" x="55.88" y="30.48"/>
+<instance part="MIX_OUT" gate="G$1" x="109.22" y="55.88" rot="R270"/>
+<instance part="TIP" gate="G$1" x="132.08" y="33.02" rot="R180"/>
+<instance part="TEST_GND" gate="G$1" x="-38.1" y="71.12"/>
+<instance part="GND8" gate="1" x="-38.1" y="68.58"/>
+<instance part="TEST_GND1" gate="G$1" x="-50.8" y="71.12"/>
+<instance part="GND9" gate="1" x="-50.8" y="68.58"/>
 </instances>
 <busses>
@@
 <wire x1="132.08" y1="53.34" x2="134.62" y2="53.34" width="0.1524" layer="91"/>
 </segment>
+<segment>
+<pinref part="TEST_GND" gate="G$1" pin="P$1"/>
+<pinref part="GND8" gate="1" pin="GND"/>
+</segment>
+<segment>
+<pinref part="TEST_GND1" gate="G$1" pin="P$1"/>
+<pinref part="GND9" gate="1" pin="GND"/>
+</segment>
 </net>
 <net name="N$9" class="0">
@@
 <pinref part="C3" gate="G$1" pin="2"/>
 <pinref part="LMG" gate="G$1" pin="1"/>
-<wire x1="63.5" y1="53.34" x2="60.96" y2="60.96" width="0.1524" layer="91"/>
+<wire x1="66.04" y1="53.34" x2="60.96" y2="60.96" width="0.1524" layer="91"/>
 </segment>
 </net>
@@
 <pinref part="C4" gate="G$1" pin="2"/>
 <pinref part="RMG" gate="G$1" pin="1"/>
-<wire x1="63.5" y1="30.48" x2="60.96" y2="38.1" width="0.1524" layer="91"/>
+<wire x1="66.04" y1="30.48" x2="60.96" y2="38.1" width="0.1524" layer="91"/>
 </segment>
 </net>
@@
 <pinref part="U$1" gate="G$1" pin="WIPER"/>
 <pinref part="C3" gate="G$1" pin="1"/>
+<wire x1="55.88" y1="53.34" x2="53.34" y2="53.34" width="0.1524" layer="91"/>
+<pinref part="LEFT_OUT" gate="G$1" pin="P$1"/>
+<junction x="55.88" y="53.34"/>
 </segment>
 </net>
@@
 <pinref part="U$2" gate="G$1" pin="WIPER"/>
 <pinref part="C4" gate="G$1" pin="1"/>
+<wire x1="55.88" y1="30.48" x2="53.34" y2="30.48" width="0.1524" layer="91"/>
+<pinref part="RIGHT_OUT" gate="G$1" pin="P$1"/>
+<junction x="55.88" y="30.48"/>
 </segment>
 </net>
@@
 <segment>
 <wire x1="109.22" y1="73.66" x2="109.22" y2="66.04" width="0.1524" layer="91"/>
-<wire x1="109.22" y1="66.04" x2="109.22" y2="53.34" width="0.1524" layer="91"/>
+<wire x1="109.22" y1="66.04" x2="109.22" y2="55.88" width="0.1524" layer="91"/>
+<wire x1="109.22" y1="55.88" x2="109.22" y2="53.34" width="0.1524" layer="91"/>
 <wire x1="93.98" y1="53.34" x2="109.22" y2="53.34" width="0.1524" layer="91"/>
 <pinref part="IC1" gate="C" pin="OUT"/>
@@
 <pinref part="COUT" gate="G$1" pin="1"/>
 <wire x1="109.22" y1="33.02" x2="114.3" y2="33.02" width="0.1524" layer="91"/>
+<pinref part="MIX_OUT" gate="G$1" pin="P$1"/>
+<junction x="109.22" y="55.88"/>
 </segment>
 </net>
@@
 <wire x1="2.54" y1="71.12" x2="0" y2="71.12" width="0.1524" layer="91"/>
 <label x="0" y="71.12" size="1.27" layer="95" rot="R90" xref="yes"/>
+<pinref part="LEFT_IN" gate="G$1" pin="P$1"/>
+<junction x="2.54" y="71.12"/>
 </segment>
 <segment>
@@
 <wire x1="2.54" y1="48.26" x2="0" y2="48.26" width="0.1524" layer="91"/>
 <label x="0" y="48.26" size="1.27" layer="95" rot="R270" xref="yes"/>
+<pinref part="RIGHT_IN" gate="G$1" pin="P$1"/>
+<junction x="2.54" y="48.26"/>
 </segment>
 <segment>
@@
 <wire x1="124.46" y1="33.02" x2="129.54" y2="33.02" width="0.1524" layer="91"/>
 <pinref part="U$4" gate="G$1" pin="RING"/>
-<wire x1="129.54" y1="33.02" x2="134.62" y2="33.02" width="0.1524" layer="91"/>
+<wire x1="129.54" y1="33.02" x2="132.08" y2="33.02" width="0.1524" layer="91"/>
+<wire x1="132.08" y1="33.02" x2="134.62" y2="33.02" width="0.1524" layer="91"/>
 <wire x1="134.62" y1="48.26" x2="129.54" y2="48.26" width="0.1524" layer="91"/>
 <wire x1="129.54" y1="48.26" x2="129.54" y2="33.02" width="0.1524" layer="91"/>
 <junction x="129.54" y="33.02"/>
-</segment>
-</net>
+<pinref part="TIP" gate="G$1" pin="P$1"/>
+<junction x="132.08" y="33.02"/>
+</segment>
+</net>
